Commit message: Created the Gazebo tutorial.

File: intro2ros/workspaces/intro2ros/src/turret_bot/urdf/turret_bot.urdf (robot description, URDF)
Before this commit: robot turret_bot, 3 links, 2 joints
Links:
- link base: mass None -> 16; geometry collision mesh filename=package://turret_bot/meshes/base.stl scale=1 1 1; visual mesh filename=package://turret_bot/meshes/base.stl scale=1 1 1
- link rotor: mass None -> 2.114; geometry collision mesh filename=package://turret_bot/meshes/rotor.stl scale=1 1 1; visual mesh filename=package://turret_bot/meshes/rotor.stl scale=1 1 1
- link slider: mass None -> 9.8075; geometry collision mesh filename=package://turret_bot/meshes/slider.stl scale=1 1 1; visual mesh filename=package://turret_bot/meshes/slider.stl scale=1 1 1

Commit message: ROS Control tutorial done.

File: intro2ros/workspaces/intro2ros/src/turret_bot/urdf/turret_bot.urdf (robot description, URDF)
Before this commit: robot turret_bot, 3 links, 2 joints
Joints:
- joint j2: limit lower=-3.141592 upper=3.141592 effort=1000 velocity=50 -> lower=-3.14 upper=3.14 effort=1000 velocity=50
